Commit message: feat: add proxsuite QP solver

File: src/guppy_description/urdf/guppy.urdf (robot description, URDF)
Before this commit: robot guppytest1, 9 links, 8 joints
Joints:
- joint thruster0C_joint: limit (none) -> lower=0 upper=0 effort=0 velocity=9999; type fixed -> revolute
- joint thruster0M_joint: limit (none) -> lower=0 upper=0 effort=0 velocity=9999; type fixed -> revolute

Commit message: feat: start to move guppy urdf to this repo

File: src/guppy_description/urdf/guppy.urdf (robot description, URDF)
Before this commit: robot guppytest1, 9 links, 8 joints
Links:
- added link cam_fl_link, mass 0; collision box size=0.06 0.03 0.03; visual box size=0.06 0.03 0.03
- added link cam_fl_optical_frame
- added link cam_fr_link, mass 0; collision box size=0.06 0.03 0.03; visual box size=0.06 0.03 0.03
- added link cam_fr_optical_frame
- added link cam_rl_link, mass 0; collision box size=0.06 0.03 0.03; visual box size=0.06 0.03 0.03
- added link cam_rl_optical_frame
- added link cam_rr_link, mass 0; collision box size=0.06 0.03 0.03; visual box size=0.06 0.03 0.03
- added link cam_rr_optical_frame
- added link camera_link, mass 0; collision box size=0.10 0.06 0.04; visual box size=0.10 0.06 0.04
- added link camera_optical_frame
- added link dvl_link, mass 0; collision box size=0.03 0.03 0.03; visual box size=0.03 0.03 0.03
- added link imu_link, mass 0; collision box size=0.01 0.01 0.01; visual box size=0.01 0.01 0.01
- link base_link: mass 12.294 -> 20; geometry collision mesh filename=package://gncea_description/meshes/base_link.STL; visual mesh filename=package://gncea_description/meshes/base_link.STL
- link thruster0C_link: mass 0.17277 -> 0; geometry collision mesh filename=package://gncea_description/meshes/thruster0C_link.STL; visual mesh filename=package://gncea_description/meshes/thruster0C_link.STL
- link thruster0M_link: mass 0.17279 -> 0; geometry collision mesh filename=package://gncea_description/meshes/thruster0M_link.STL; visual mesh filename=package://gncea_description/meshes/thruster0M_link.STL
- link thruster1C_link: mass 0.17277 -> 0; geometry collision mesh filename=package://gncea_description/meshes/thruster1C_link.STL; visual mesh filename=package://gncea_description/meshes/thruster1C_link.STL
- link thruster1M_link: mass 0.17279 -> 0; geometry collision mesh filename=package://gncea_description/meshes/thruster1M_link.STL; visual mesh filename=package://gncea_description/meshes/thruster1M_link.STL
- link thruster2C_link: mass 0.17277 -> 0; geometry collision mesh filename=package://gncea_description/meshes/thruster2C_link.STL; visual mesh filename=package://gncea_description/meshes/thruster2C_link.STL
- link thruster2M_link: mass 0.17279 -> 0; geometry collision mesh filename=package://gncea_description/meshes/thruster2M_link.STL; visual mesh filename=package://gncea_description/meshes/thruster2M_link.STL
- link thruster3C_link: mass 0.17277 -> 0; geometry collision mesh filename=package://gncea_description/meshes/thruster3C_link.STL; visual mesh filename=package://gncea_description/meshes/thruster3C_link.STL
- link thruster3M_link: mass 0.17277 -> 0; geometry collision mesh filename=package://gncea_description/meshes/thruster3M_link.STL; visual mesh filename=package://gncea_description/meshes/thruster3M_link.STL
Joints:
- added joint cam_fl_joint: type fixed, parent base_link, child cam_fl_link, origin xyz=0.25 0.18 0.10 rpy=0 0 0.78539816339
- added joint cam_fl_optical_joint: type fixed, parent cam_fl_link, child cam_fl_optical_frame, origin xyz=0 0 0 rpy=-1.57079632679 0 -1.57079632679
- added joint cam_fr_joint: type fixed, parent base_link, child cam_fr_link, origin xyz=0.25 -0.18 0.10 rpy=0 0 -0.78539816339
- added joint cam_fr_optical_joint: type fixed, parent cam_fr_link, child cam_fr_optical_frame, origin xyz=0 0 0 rpy=-1.57079632679 0 -1.57079632679
- added joint cam_rl_joint: type fixed, parent base_link, child cam_rl_link, origin xyz=-0.25 0.18 0.10 rpy=0 0 2.35619449019
- added joint cam_rl_optical_joint: type fixed, parent cam_rl_link, child cam_rl_optical_frame, origin xyz=0 0 0 rpy=-1.57079632679 0 -1.57079632679
- added joint cam_rr_joint: type fixed, parent base_link, child cam_rr_link, origin xyz=-0.25 -0.18 0.10 rpy=0 0 -2.35619449019
- added joint cam_rr_optical_joint: type fixed, parent cam_rr_link, child cam_rr_optical_frame, origin xyz=0 0 0 rpy=-1.57079632679 0 -1.57079632679
- added joint camera_joint: type fixed, parent base_link, child camera_link, origin xyz=0.00 0.20 0.10 rpy=0 0 1.57079632679
- added joint camera_optical_joint: type fixed, parent camera_link, child camera_optical_frame, origin xyz=0 0 0 rpy=-1.57079632679 0 1.57079632679
- added joint dvl_joint: type fixed, parent base_link, child dvl_link, origin xyz=0.0 0.0 -0.05 rpy=0 0 0
- added joint imu_joint: type fixed, parent base_link, child imu_link, origin xyz=0 0 0.05 rpy=0 0 0
- joint thruster0C_joint: limit lower=0 upper=0 effort=0 velocity=9999 -> (none); type revolute -> fixed
- joint thruster0M_joint: limit lower=0 upper=0 effort=0 velocity=9999 -> (none); origin xyz=0.2903 -2.5E-05 -0.013798 rpy=1.5708 1.5708 -1.5708 -> xyz=0.2903 0 -0.013798 rpy=1.5708 1.5708 -1.5708; type revolute -> fixed
- joint thruster1M_joint: origin xyz=-2.5E-05 -0.2649 -0.013798 rpy=0 1.5708 -1.5708 -> xyz=0 -0.2649 -0.013798 rpy=0 1.5708 -1.5708
- joint thruster2M_joint: origin xyz=-0.2903 2.5E-05 -0.013798 rpy=1.5708 1.5708 -1.5708 -> xyz=-0.2903 0 -0.013798 rpy=1.5708 1.5708 -1.5708
- joint thruster3M_joint: origin xyz=2.5E-05 0.2649 -0.013798 rpy=3.1416 1.5708 -1.5708 -> xyz=0 0.2649 -0.013798 rpy=3.1416 1.5708 -1.5708

Commit message: feat: add urdf changes

File: src/guppy_description/urdf/guppy.urdf (robot description, URDF)
Before this commit: robot guppytest1, 21 links, 20 joints
Links:
- link base_link: geometry collision mesh filename=package://guppy_description/meshes/base_link.STL; visual mesh filename=package://guppy_description/meshes/base_link.STL
- link thruster0C_link: geometry collision mesh filename=package://guppy_description/meshes/thruster0C_link.STL; visual mesh filename=package://guppy_description/meshes/thruster0C_link.STL
- link thruster0M_link: geometry collision mesh filename=package://guppy_description/meshes/thruster0M_link.STL; visual mesh filename=package://guppy_description/meshes/thruster0M_link.STL
- link thruster1C_link: geometry collision mesh filename=package://guppy_description/meshes/thruster1C_link.STL; visual mesh filename=package://guppy_description/meshes/thruster1C_link.STL
- link thruster1M_link: geometry collision mesh filename=package://guppy_description/meshes/thruster1M_link.STL; visual mesh filename=package://guppy_description/meshes/thruster1M_link.STL
- link thruster2C_link: geometry collision mesh filename=package://guppy_description/meshes/thruster2C_link.STL; visual mesh filename=package://guppy_description/meshes/thruster2C_link.STL
- link thruster2M_link: geometry collision mesh filename=package://guppy_description/meshes/thruster2M_link.STL; visual mesh filename=package://guppy_description/meshes/thruster2M_link.STL
- link thruster3C_link: geometry collision mesh filename=package://guppy_description/meshes/thruster3C_link.STL; visual mesh filename=package://guppy_description/meshes/thruster3C_link.STL
- link thruster3M_link: geometry collision mesh filename=package://guppy_description/meshes/thruster3M_link.STL; visual mesh filename=package://guppy_description/meshes/thruster3M_link.STL

Commit message: FCS

File: src/guppy_description/urdf/guppy.urdf (robot description, URDF)
Before this commit: robot guppytest1, 21 links, 20 joints
Links:
- added link FCS_camera_link, mass 0; collision box size=0.06 0.03 0.03; visual box size=0.06 0.03 0.03
- added link FCS_camera_optical_frame
Joints:
- added joint FCS_camera_joint: type fixed, parent base_link, child FCS_camera_link, origin xyz=0.30 0.0 0.05 rpy=0 0 0
- added joint FCS_camera_optical_joint: type fixed, parent FCS_camera_link, child FCS_camera_optical_frame, origin xyz=0 0 0 rpy=-1.57079632679 0 -1.57079632679

Commit message: chore: dvl and imu edits

File: src/guppy_description/urdf/guppy.urdf (robot description, URDF)
Before this commit: robot guppytest1, 21 links, 20 joints
Joints:
- joint dvl_joint: origin xyz=0.0 0.0 -0.05 rpy=0 0 0 -> xyz=-0.2 0.0 -0.125 rpy=0 0 0
- joint imu_joint: origin xyz=0 0 0.05 rpy=0 0 0 -> xyz=0.22 0.0625 0.125 rpy=0 0 0

Commit message: fix: add many integration changes

File: src/guppy_description/urdf/guppy.urdf (robot description, URDF)
Before this commit: robot guppytest1, 21 links, 20 joints
Links:
- removed link imu_link
- added link vectornav, mass 0; collision box size=0.01 0.01 0.01; visual box size=0.01 0.01 0.01
Joints:
- joint imu_joint: child imu_link -> vectornav

Commit message: feat: late night pid tuning

File: src/guppy_description/urdf/guppy.urdf (robot description, URDF)
Before this commit: robot guppytest1, 21 links, 20 joints
Joints:
- joint imu_joint: origin xyz=0.22 0.0625 0.125 rpy=0 0 0 -> xyz=0.22 0.0625 0.125 rpy=0 0 -1.570796326

Commit message: feat: add slam

File: src/guppy_description/urdf/guppy.urdf (robot description, URDF)
Before this commit: robot guppytest1, 21 links, 20 joints
Links:
- added link test, mass 0; collision box size=0.06 0.03 0.03; visual box size=0.06 0.03 0.03
Joints:
- added joint test_joint: type fixed, parent base_link, child test, origin xyz=-0.10 +0.15 0.4 rpy=0 0 1.579
